Commit message: Better urdf of platform robot

File: urdf/platform.xacro (robot description, xacro)
@@ -3,4 +3,5 @@
   <!-- Include all xacro:macro definition files -->
   <xacro:include filename="$(find platform_description)/urdf/properties.xacro" />
+  <xacro:include filename="$(find platform_description)/urdf/mast.xacro" />
   <gazebo>
     <plugin
@@ -126,5 +127,6 @@
     <child link="left_wheel"/>
     <axis xyz="0 0 1"/>
-    <limit lower="-1.79769e+308" upper="1.79769e+308" effort="10" velocity="20" />
+    <dynamics damping="0.15"/>
+    <limit lower="-1.79769e+308" upper="1.79769e+308" effort="35.8" velocity="100" />
   </joint>
   <joint name="right_wheel_joint" type="revolute">
@@ -133,5 +135,6 @@
     <child link="right_wheel"/>
     <axis xyz="0 0 1"/>
-    <limit lower="-1.79769e+308" upper="1.79769e+308" effort="10" velocity="20" />
+    <dynamics damping="0.15"/>
+    <limit lower="-1.79769e+308" upper="1.79769e+308" effort="35.8" velocity="100" />
   </joint>
   <xacro:if value="${wheel_number == 4}">
@@ -277,4 +280,34 @@
    </joint>
   </xacro:if>
+    <!-- MAST -->
+  <!-- <link name="mast">
+    <visual>
+        <origin xyz="0.0 0.0 ${mast_height/2}" rpy="0 0 0" />
+        <geometry>
+          <cylinder length="${mast_height}" radius="${wheel_radius}"/>
+        </geometry>
+        <material name="blue">
+          <color rgba="0 1 0 1"/>
+        </material>
+    </visual>
+    <collision>
+      <origin xyz="0.0 0.0 ${mast_height/2}" rpy="0 0 0" />
+      <geometry>
+        <cylinder length="${mast_height}" radius="${wheel_radius}"/>
+      </geometry>
+    </collision>
+<     <inertial>
+      <origin xyz="0.0 0.0 ${mast_height/2}" rpy="0 0 0" />
+      <xacro:cylinder_inertia  m="20" r="${wheel_radius}" h="${mast_height}" />
+    </inertial> >
+  </link>
+  <joint name="mast_joint" type="fixed">
+    <origin xyz="0 0 ${base_height + 0.05/2 + base_ground_clearance/2.0}" rpy="0 0 0" />
+    <parent link="base_footprint"/>
+    <child link="mast" />
+  </joint> -->
+  <xacro:Mast name="mast" parent="base_footprint" >
+    <origin rpy="0.0 0.0 0.0" xyz="0.0 0.0 ${base_height}" />
+  </xacro:Mast>
   <gazebo>
     <plugin
@@ -291,6 +324,6 @@
       <frame_id>odom</frame_id>
       <child_frame_id>base_footprint</child_frame_id>
-      <max_acceleration>1</max_acceleration>
-      <max_velocity>1.3</max_velocity>
+      <max_acceleration>100</max_acceleration>
+      <max_velocity>2</max_velocity>
     </plugin>
   </gazebo>

File: urdf/properties.xacro (robot description, xacro)
@@ -13,19 +13,21 @@
     <!-- Main body radius and height -->
     <!-- Main Body Cylinder base   -->
-    <xacro:property name="base_height" value="0.15" />
-    <xacro:property name="base_radius" value="0.26" />
-    <xacro:property name="base_ground_clearance" value="0.1" />
-    <xacro:property name="base_mass" value="40" /> <!-- in kg-->
+    <xacro:property name="base_height" value="0.36" />
+    <xacro:property name="base_length" value="1.689" />
+    <xacro:property name="base_radius" value="0.641" />
+    <xacro:property name="base_ground_clearance" value="0.2" />
+    <xacro:property name="base_mass" value="250" /> <!-- in kg-->
     <xacro:property name="base_shape" value="rectangle" /> <!-- circle, rectangle-->
     <!-- Casters -->
-    <xacro:property name="caster_radius" value="0.05" />
+    <xacro:property name="caster_radius" value="0.075" />
     <xacro:property name="caster_mass" value="0.2" />
     <!-- Wheels -->
-    <xacro:property name="wheel_radius" value="0.075" />
-    <xacro:property name="wheel_height" value="0.02" />
+    <xacro:property name="wheel_radius" value="0.125" />
+    <xacro:property name="wheel_height" value="0.04" />
     <xacro:property name="wheel_number" value="6" />
-    <xacro:property name="wheel_mass" value="1.0" /> <!-- in kg-->
+    <xacro:property name="wheel_mass" value="3.0" /> <!-- in kg-->
     <xacro:property name="base_x_origin_to_wheel_origin" value="0.0" />
-    <xacro:property name="base_y_origin_to_wheel_origin" value="0.235" />
+    <xacro:property name="base_y_origin_to_wheel_origin" value="${0.944/2}" />
+    <xacro:property name="mast_height" value="12" />
     <!-- SENSORS -->
     <!-- laser sensors -->
